File: 4_Schematics and Boards Layout/4_6_Schematics/MainBoard/RADAR_Main_Board_2.kicad_sch (KiCad schematic)
At the start: 130 parts, among them J1 142-0731-211, J18 142-0731-211, J19 CJT-T-P-HH-ST-TH1, U2 STM32F746ZGT7, U42 XC7A50T-2FTG256I, U6 FT601Q-B-T, U9 MT25QL01GBBB8E12-0AUT, X53 MINI-USB-32005-201

Commit message: KiCad FPGA swap schematic wiring + MCU scan scheduler fix
Manual KiCad work: FPGA swap from XC7A100T to XC7A200T on MainBoard
schematic — rewiring U42 connections, ERC fixes, power rail updates,
PCB footprint swap. Includes backup files and automation scripts.

MCU: scan scheduler contract test + main.cpp updates.
Parts:
- removed R12, R2, R3, R9: 100R, RADAR_Main_Board:R0201, symbol RADAR_Main_Board-eagle-import:RR0201
- removed R138, R139, R140, R144: 1k, RADAR_Main_Board:R0201, symbol RADAR_Main_Board-eagle-import:RR0201
- removed R141, R142: 4.7k, RADAR_Main_Board:R0201, symbol RADAR_Main_Board-eagle-import:RR0201
- removed R145, R146, R60, R61, R83, R84: 33R, RADAR_Main_Board:R0201, symbol RADAR_Main_Board-eagle-import:RR0201
- removed U42: XC7A50T-2FTG256I, RADAR_Main_Board:BGA256C100P16X16_1700X1700X155, symbol RADAR_Main_Board-eagle-import:XC7A50T-2FTG256I
- added R12, R138, R139, R140, R141, R142, R144, R145, R146, R177, R178, R179, R180, R181, R182, R183, R184, R185, R186, R187, R188, R189, R190, R191, R192, R2, R3, R60, R61, R83, R84, R9: 33R, RADAR_Main_Board:R0402, symbol RADAR_Main_Board-eagle-import:RR0402
- added R174, R175, R176: 4.7k, RADAR_Main_Board:R0201, symbol RADAR_Main_Board-eagle-import:RR0201
- added U42: XC7A200T-FBG484I, symbol FPGA_Xilinx_Artix7:XC7A200T-FBG484
- JP3: footprint RADAR_Main_Board:2X04 -> Connector_PinHeader_1.00mm:PinHeader_2x04_P1.00mm_Vertical_SMD
- R6: value 100R -> 300R
Connections:
- net +1V0_FPGA: now also U42.H10 (VCCINT), U42.H8 (VCCINT), U42.J11 (VCCBRAM), U42.J7 (VCCINT), U42.J9 (VCCINT), U42.K8 (VCCINT), U42.L11 (VCCBRAM), U42.L7 (VCCINT), U42.M8 (VCCINT), U42.N11 (VCCBRAM), U42.N7 (VCCINT), U42.P10 (VCCINT), U42.P8 (VCCINT), U42.R7 (VCCINT), U42.R9 (VCCINT), U42.T10 (VCCINT), U42.T8 (VCCINT)
- net +1V8_FPGA: now also R143.2, R6.1, R174.2, R176.2, U42.AA7 (VCCO_34), U42.AB4 (VCCO_34), U42.C1 (VCCO_35), U42.E12 (VCCBATT_0), U42.F12 (VCCO_0), U42.F2 (VCCO_35), U42.H12 (VCCAUX), U42.H6 (VCCO_35), U42.J3 (VCCO_35), U42.K10 (VCCADC_0), U42.K12 (VCCAUX), U42.M12 (VCCAUX), U42.M4 (VCCO_35), U42.N1 (VCCO_35), U42.P12 (VCCAUX), U42.R11 (VCCAUX), U42.R5 (VCCO_34), U42.T12 (VCCO_0), U42.T2 (VCCO_34), U42.U8 (CFGBVS_0), U42.V6 (VCCO_34), U42.W3 (VCCO_34)
- net +3V3_FPGA: now also R69.1, U42.A17 (VCCO_16), U42.AA17 (VCCO_13), U42.AB14 (VCCO_13), U42.B14 (VCCO_16), U42.C21 (VCCO_16), U42.D18 (VCCO_16), U42.E15 (VCCO_16), U42.F22 (VCCO_16), U42.G19 (VCCO_15), U42.H16 (VCCO_15), U42.J13 (VCCO_15), U42.K20 (VCCO_15), U42.L17 (VCCO_15), U42.M14 (VCCO_14), U42.N21 (VCCO_15), U42.P18 (VCCO_14), U42.R15 (VCCO_14), U42.T22 (VCCO_14), U42.U19 (VCCO_14), U42.V16 (VCCO_13), U42.W13 (VCCO_13), U42.Y10 (VCCO_13), U42.Y20 (VCCO_14); no longer R143.2, R69.2
- net ADAR_1_CS_1V8: now also U42.Y2 (IO_L4N_T0_34)
- net ADAR_1_CS_3V3: now also U42.M22 (IO_L15N_T2_DQS_ADV_B_15)
- net ADAR_2_CS_1V8: now also U42.W2 (IO_L4P_T0_34)
- net ADAR_2_CS_3V3: now also U42.N22 (IO_L15P_T2_DQS_15)
- net ADAR_3_CS_1V8: now also U42.R2 (IO_L3N_T0_DQS_34)
- net ADAR_3_CS_3V3: now also U42.L20 (IO_L14N_T2_SRCC_15)
- net ADAR_4_CS_1V8: now also U42.R3 (IO_L3P_T0_DQS_34)
- net ADAR_4_CS_3V3: now also U42.L19 (IO_L14P_T2_SRCC_15)
- net ADAR_RX_LOAD_1: now also U42.AA5 (IO_L10P_T1_34)
- net ADAR_RX_LOAD_2: now also U42.AB1 (IO_L7N_T1_34)
- net ADAR_RX_LOAD_3: now also U42.AB2 (IO_L8N_T1_34)
- net ADAR_RX_LOAD_4: now also U42.AA3 (IO_L9N_T1_DQS_34)
- net ADAR_TR_1: now also U42.U1 (IO_L1N_T0_34)
- net ADAR_TR_2: now also U42.T1 (IO_L1P_T0_34)
- net ADAR_TR_3: now also U42.T3 (IO_0_34)
- net ADAR_TR_4: now also U42.Y1 (IO_L5N_T0_34)
- net ADAR_TX_LOAD_1: now also U42.AB5 (IO_L10N_T1_34)
- net ADAR_TX_LOAD_2: now also U42.AA1 (IO_L7P_T1_34)
- net ADAR_TX_LOAD_3: now also U42.AB3 (IO_L8P_T1_34)
- net ADAR_TX_LOAD_4: now also U42.Y3 (IO_L9P_T1_DQS_34)
- net ADC_D0_N: now also U42.V22 (IO_L3N_T0_DQS_EMCCLK_14)
- net ADC_D0_P: now also U42.T21 (IO_L4P_T0_D04_14)
- net ADC_D1_N: now also U42.R21 (IO_L2N_T0_D03_14)
- net ADC_D1_P: now also U42.U22 (IO_L3P_T0_DQS_PUDC_B_14)
- net ADC_D2_N: now also U42.R22 (IO_L1N_T0_D01_DIN_14); no longer R6.1
- net ADC_D2_P: now also U42.P21 (IO_L2P_T0_D02_14); no longer R6.2
- net ADC_D3_N: now also U42.T18 (IO_L20N_T3_A07_D23_14); no longer R5.1
- net ADC_D3_P: now also U42.N17 (IO_L21P_T3_DQS_14); no longer R5.2
- net ADC_D4_N: now also U42.R14 (IO_L19N_T3_A09_D25_VREF_14); no longer R7.1
- net ADC_D4_P: now also U42.R18 (IO_L20P_T3_A08_D24_14); no longer R7.2
- net ADC_D5_N: now also U42.V19 (IO_L14N_T2_SRCC_14)
- net ADC_D5_P: now also U42.AA19 (IO_L15P_T2_DQS_RDWR_B_14)
- net ADC_D6_N: now also U42.AB20 (IO_L15N_T2_DQS_DOUT_CSO_B_14); no longer R8.1
- net ADC_D6_P: now also U42.V17 (IO_L16P_T2_CSI_B_14); no longer R8.2
- net ADC_D7_N: now also R11.1; no longer R10.1
- net ADC_D7_P: now also U42.Y18 (IO_L13P_T2_MRCC_14); no longer R10.2
- net ADC_DCO_N: now also R10.2, U42.W20 (IO_L12N_T1_MRCC_14)
- net ADC_DCO_P: now also R10.1, U42.W19 (IO_L12P_T1_MRCC_14)
- net ADC_OR_N: now also U42.AB18 (IO_L17N_T2_A13_D29_14); no longer R11.1
- net ADC_OR_P: now also U42.U17 (IO_L18P_T2_A12_D28_14); no longer R11.2
- net ADC_PWRD: now also U42.Y19 (IO_L13N_T2_MRCC_14)
- net DAC_0: now also U42.G18 (IO_L4N_T0_15)
- net DAC_1: now also U42.J15 (IO_L5P_T0_AD9P_15)
- net DAC_2: now also U42.H18 (IO_L6N_T0_VREF_15)
- net DAC_3: now also U42.H22 (IO_L7N_T1_AD2N_15)
- net DAC_4: now also U42.H20 (IO_L8P_T1_AD10P_15)
- net DAC_5: now also U42.G20 (IO_L8N_T1_AD10N_15)
- net DAC_6: now also U42.K22 (IO_L9N_T1_DQS_AD3N_15)
- net DAC_7: now also U42.M21 (IO_L10P_T1_AD11P_15)
- net DAC_SLEEP: now also U42.G16 (IO_L2N_T0_AD8N_15)
- net DIG_0: now also U42.L13 (IO_L20N_T3_A19_15)
- net DIG_1: now also U42.M13 (IO_L20P_T3_A20_15)
- net DIG_2: now also U42.K14 (IO_L19N_T3_A21_VREF_15)
- net DIG_3: now also U42.K13 (IO_L19P_T3_A22_15)
- net DIG_4: now also U42.M20 (IO_L18N_T2_A23_15)
- net DIG_5: now also U42.N20 (IO_L18P_T2_A24_15)
- net DIG_6: now also U42.N19 (IO_L17N_T2_A25_15)
- net DIG_7: now also U42.N18 (IO_L17P_T2_A26_15)
- net FPGA_ADC_CLOCK_N: now also U42.N14 (IO_L23N_T3_A02_D18_14)
- net FPGA_ADC_CLOCK_P: now also U42.P16 (IO_L24P_T3_A01_D17_14)
- net FPGA_CLOCK_TEST: now also U42.K18 (IO_L13P_T2_MRCC_15)
- net FPGA_DAC_CLOCK: now also U42.G21 (IO_L24P_T3_16)
- net FPGA_FLASH_CLK: now also U42.L12 (CCLK_0)
- net FPGA_FLASH_DQ0: now also U42.U20 (IO_L11P_T1_SRCC_14)
- net FPGA_FLASH_DQ1: now also U42.AB22 (IO_L10N_T1_D15_14)
- net FPGA_FLASH_DQ2: now also U42.AB21 (IO_L10P_T1_D14_14)
- net FPGA_FLASH_DQ3: now also U42.Y22 (IO_L9N_T1_DQS_D13_14)
- net FPGA_FLASH_NCS: now also U42.T19 (IO_L6P_T0_FCS_B_14)
- net FPGA_FLASH_NRST: now also U42.T20 (IO_L6N_T0_D08_VREF_14)
- net FPGA_PUDC_B: now also R69.2, U42.Y21 (IO_L9P_T1_DQS_14); no longer R69.1
- net FPGA_SYS_CLOCK: now also U42.M15 (IO_L24P_T3_RS1_15)
- net FPGA_TCK: now also U42.V12 (TCK_0)
- net FPGA_TDI: now also U42.R13 (TDI_0)
- net FPGA_TDO: now also U42.U13 (TDO_0)
- net FPGA_TMS: now also U42.T13 (TMS_0)
- net GND: now also U6.1 (GND_2), U6.26 (GND_3), U6.29 (GND_4), U6.36 (GND_5), U6.77 (GND), R175.2, U42.A11 (GND), U42.A12 (GND), U42.A2 (GND), U42.A22 (GND), U42.A3 (GND), U42.A5 (GND), U42.A7 (GND), U42.A9 (GND), U42.AA12 (GND), U42.AA2 (GND), U42.AA22 (GND), U42.AB19 (GND), U42.AB9 (GND), U42.B12 (GND), U42.B19 (GND), U42.B3 (GND), U42.C10 (GND), U42.C12 (GND), U42.C16 (GND), U42.C3 (GND), U42.C6 (GND), U42.D12 (GND), U42.D13 (GND), U42.D3 (GND), U42.D4 (GND), U42.D8 (GND), U42.E11 (GND), U42.E20 (GND), U42.E4 (GND), U42.E5 (GND), U42.E7 (GND), U42.E9 (GND), U42.F11 (GND), U42.F17 (GND), U42.F5 (GND), U42.G10 (GND), U42.G12 (GND), U42.G14 (GND), U42.G5 (GND), U42.G6 (GND), U42.G7 (GND), U42.G8 (GND), U42.G9 (GND), U42.H1 (GND), U42.H11 (GND), U42.H21 (GND), U42.H7 (GND), U42.H9 (GND), U42.J10 (GND), U42.J12 (GND), U42.J18 (GND), U42.J8 (GND), U42.K11 (GND), U42.K15 (GND), U42.K5 (GND), U42.K7 (GND), U42.K9 (GNDADC_0), U42.L2 (GND), U42.L22 (GND), U42.L8 (GND), U42.L9 (VREFN_0), U42.M11 (GND), U42.M19 (GND), U42.M7 (GND), U42.N16 (GND), U42.N6 (GND), U42.N8 (GND), U42.P11 (GND), U42.P13 (GND), U42.P3 (GND), U42.P7 (GND), U42.P9 (GND), U42.R10 (GND), U42.R12 (GND), U42.R20 (GND), U42.R8 (GND), U42.T11 (GND), U42.T17 (GND), U42.T7 (GND), U42.T9 (GND), U42.U14 (GND), U42.U4 (GND), U42.V1 (GND), U42.V11 (GND), U42.V21 (GND), U42.W18 (GND), U42.W8 (GND), U42.Y15 (GND), U42.Y5 (GND)
- net M3S_VCTRL: now also U42.G15 (IO_L2P_T0_AD8P_15)
- net MIX_RX_EN: now also U42.L15 (IO_L22N_T3_A16_15)
- net MIX_TX_EN: now also U42.H13 (IO_L1P_T0_AD0P_15)
- net STM32_MISO1: now also U42.M18 (IO_L16P_T2_A28_15)
- net STM32_MISO_1V8: now also U42.U2 (IO_L2P_T0_34)
- net STM32_MOSI1: now also U42.L18 (IO_L16N_T2_A27_15)
- net STM32_MOSI_1V8: now also U42.V2 (IO_L2N_T0_34)
- net STM32_SCLK1: now also U42.K19 (IO_L13N_T2_MRCC_15)
- net STM32_SCLK_1V8: now also U42.U3 (IO_L6P_T0_34)
- net at R143.1: now also U42.U12 (INIT_B_0)
- net FPGA-A13: now reaches U6.40 (DATA_0)
- net FPGA-A13: now also R192.1
- net FPGA-A14: now reaches U6.41 (DATA_1)
- net FPGA-A14: now also R188.1
- net FPGA-A15: now reaches U6.42 (DATA_2)
- net FPGA-A15: now also R189.1
- net FPGA-A16: now reaches U6.43 (DATA_3)
- net FPGA-A16: now also R190.1
- net FPGA-A18: now reaches U6.44 (DATA_4)
- net FPGA-A18: now also R191.1
- net FPGA-A19: now reaches U6.45 (DATA_5)
- net FPGA-A19: now also R185.1
- net FPGA-A20: now reaches U6.46 (DATA_6)
- net FPGA-A20: now also R186.1
- net FPGA-A21: now reaches U6.47 (DATA_7)
- net FPGA-A21: now also R187.1
- net FPGA-B13: now reaches U6.50 (DATA_8)
- net FPGA-B13: now also R2.1
- net FPGA-B15: now reaches U6.51 (DATA_9)
- net FPGA-B15: now also R3.1
- net FPGA-B16: now reaches U6.52 (DATA_10)
- net FPGA-B16: now also R9.1
- net FPGA-B17: now reaches U6.53 (DATA_11)
- net FPGA-B17: now also R12.1
- net FPGA-B18: now reaches U6.54 (DATA_12)
- net FPGA-B18: now also R60.1
- net FPGA-B20: now reaches U6.55 (DATA_13)
- net FPGA-B20: now also R61.1
- net FPGA-B21: now reaches U6.56 (DATA_14)
- net FPGA-B21: now also R83.1
- net FPGA-B22: now reaches U6.57 (DATA_15)
- net FPGA-B22: now also R84.1
- net FPGA-D14: now reaches U6.60 (DATA_16)
- net FPGA-D14: now also R177.1
- net FPGA-D15: now reaches U6.61 (DATA_17)
- net FPGA-D15: now also R178.1
- net FPGA-D16: now reaches U6.62 (DATA_18)
- net FPGA-D16: now also R179.1
- net FPGA-D17: now reaches U6.63 (DATA_19)
- net FPGA-D17: now also R180.1
- net FPGA-D19: now reaches U6.64 (DATA_20)
- net FPGA-D19: now also R181.1
- net FPGA-D20: now reaches U6.65 (DATA_21)
- net FPGA-D20: now also R182.1
- net FPGA-D21: now reaches U6.66 (DATA_22)
- net FPGA-D21: now also R183.1
- net FPGA-D22: now reaches U6.67 (DATA_23)
- net FPGA-D22: now also R184.1
- net FPGA-E13: now reaches U6.69 (DATA_24)
- net FPGA-E14: now reaches U6.70 (DATA_25)
- net FPGA-E16: now reaches U6.71 (DATA_26)
- net FPGA-E17: now reaches U6.72 (DATA_27)
- net FPGA-E18: now reaches U6.73 (DATA_28)
- net FPGA-E19: now reaches U6.74 (DATA_29)
- net FPGA-E21: now reaches U6.75 (DATA_30)
- net FPGA-E22: now reaches U6.76 (DATA_31)
- new net: R175.1, U42.U10 (M1_0), U42.U9 (M2_0)
- new net: R6.2, U42.G11 (DONE_0)
- new net: R11.2, U42.P17 (IO_L21N_T3_DQS_A06_D22_14)
- new net: R176.1, U42.U11 (M0_0)
- new net: R174.1, U42.N12 (PROGRAM_B_0)
- new net FT-40: R192.2, U42.A13 (IO_L10P_T1_16)
- new net FT-41: R188.2, U42.A14 (IO_L10N_T1_16)
- new net FT-42: R189.2, U42.A15 (IO_L9P_T1_DQS_16)
- new net FT-43: R190.2, U42.A16 (IO_L9N_T1_DQS_16)
- new net FT-44: R191.2, U42.A18 (IO_L17P_T2_16)
- new net FT-45: R185.2, U42.A19 (IO_L17N_T2_16)
- new net FT-46: R186.2, U42.A20 (IO_L16N_T2_16)
- new net FT-47: R187.2, U42.A21 (IO_L21N_T3_DQS_16)
- new net FT-50: R2.2, U42.B13 (IO_L8N_T1_16)
- new net FT-51: R3.2, U42.B15 (IO_L7P_T1_16)
- new net FT-52: R9.2, U42.B16 (IO_L7N_T1_16)
- new net FT-53: R12.2, U42.B17 (IO_L11P_T1_SRCC_16)
- new net FT-54: R60.2, U42.B18 (IO_L11N_T1_SRCC_16)
- new net FT-55: R61.2, U42.B20 (IO_L16P_T2_16)
- new net FT-56: R83.2, U42.B21 (IO_L21P_T3_DQS_16)
- new net FT-57: R84.2, U42.B22 (IO_L20N_T3_16)
- new net FT-60: R177.2, U42.D14 (IO_L6P_T0_16)
- new net FT-61: R178.2, U42.D15 (IO_L6N_T0_VREF_16)
- new net FT-62: R179.2, U42.D16 (IO_L5N_T0_16)
- new net FT-63: R180.2, U42.D17 (IO_L12P_T1_MRCC_16)
- new net FT-64: R181.2, U42.D19 (IO_L14N_T2_SRCC_16)
- new net FT-65: R182.2, U42.D20 (IO_L19P_T3_16)
- new net FT-66: R183.2, U42.D21 (IO_L23N_T3_16)
- new net FT-67: R184.2, U42.D22 (IO_L22N_T3_16)
- new net FT-69: U42.E13 (IO_L4P_T0_16)
- new net FT-70: U42.E14 (IO_L4N_T0_16)
- new net FT-71: U42.E16 (IO_L5P_T0_16)
- new net FT-72: U42.E17 (IO_L2N_T0_16)
- new net FT-73: U42.E18 (IO_L15N_T2_DQS_16)
- new net FT-74: U42.E19 (IO_L14P_T2_SRCC_16)
- new net FT-75: U42.E21 (IO_L23P_T3_16)
- new net FT-76: U42.E22 (IO_L22P_T3_16)
- no-connect marks 32 -> 38
Other:
- moved on the sheet: C108, C109, C110, C111, C112, C113, C153, C154, C155, C156, C157, C158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

Commit message: FPGA v8c: BRAM playback pipeline with 2048-entry FIFO + USB pipe init fix
- Add unified playback wrapper (radar_system_top_te0713_umft601x_playback.v)
  with BRAM->DSP->USB pipeline, 2048-entry range FIFO, and 3-state
  handshake pop FSM for lossless data delivery to FT601
- Add write_idle output to usb_data_interface.v with fsm_encoding=none
  attributes to prevent Vivado FSM inference bugs
- Add _init_pipes() to radar_protocol.py and ft601_stream_server.py:
  ClearStreamPipe+SetStreamPipe sequence fixes D3XX read timeouts after
  FPGA reprogramming or USB reconnects
- Add Vivado build script, programming script, and 54-test testbench
- KiCad main board schematic wiring progress
- Verified: 2048 range packets delivered end-to-end through full pipeline
  (FPGA->FT601->USB3->stream server->TCP->SSH tunnel->GUI dashboard)
Parts:
- removed R5, R7, R8: 100R, RADAR_Main_Board:R0201, symbol RADAR_Main_Board-eagle-import:RR0201
- added C187, C189, C190, C191, C193, C194, C195, C352: 100nF, RADAR_Main_Board:C0805, symbol RADAR_Main_Board-eagle-import:C-EUC0805
- added C188, C192: 4.7uF, RADAR_Main_Board:C0805, symbol RADAR_Main_Board-eagle-import:C-EUC0805
- added R193, R194, R195, R196, R197, R198, R199, R200, R201, R202, R203: 33R, RADAR_Main_Board:R0402, symbol RADAR_Main_Board-eagle-import:RR0402
- added R204, R205: 10K, RADAR_Main_Board:R0402, symbol RADAR_Main_Board-eagle-import:RR0402
Connections:
- net +3V3_FPGA: now also R204.2, R205.2
- net AVDD: now also C187.1, C188.1
- net FPGA-E13: now also R138.1
- net FPGA-E14: now also R139.1
- net FPGA-E16: now also R140.1
- net FPGA-E17: now also R141.1
- net FPGA-E18: now also R142.1
- net FPGA-E19: now also R144.1
- net FPGA-E21: now also R145.1
- net FPGA-E22: now also R146.1
- net FT-69: now also R138.2
- net FT-70: now also R139.2
- net FT-71: now also R140.2
- net FT-72: now also R141.2
- net FT-73: now also R142.2
- net FT-74: now also R144.2
- net FT-75: now also R145.2
- net FT-76: now also R146.2
- net GND: now also C187.2, C188.2, C189.2, C190.2, C191.2, C192.2, C193.2, C194.2, C195.2, C352.2
- net VCC33: now also C193.1
- net VCC33_2: now also C190.1
- net VCCIO: now also C352.1
- net VCCIO_2: now also C189.1
- net VCCIO_3: now also C194.1
- net VCCIO_4: now also C195.1
- net VDDA: now also C191.1, C192.1
- net at U42.C13 (IO_L8P_T1_16): now also R193.1
- net at U42.C14 (IO_L3P_T0_DQS_16): now also R194.1
- net at U42.C15 (IO_L3N_T0_DQS_16): now also R195.1
- net at U42.C17 (IO_L12N_T1_MRCC_16): now also R196.1
- net at U42.C19 (IO_L13N_T2_MRCC_16): now also R201.1
- net at U42.C20 (IO_L19N_T3_VREF_16): now also R202.1
- net at U42.C22 (IO_L20P_T3_16): now also R200.1
- net at U42.F13 (IO_L1P_T0_16): now also R198.1
- net at U42.F14 (IO_L1N_T0_16): now also R197.1
- net at U42.F15 (IO_0_16): now also R199.1, R205.1
- net at U42.F16 (IO_L2P_T0_16): now also R203.1, R204.1
- net FPGA-F15: now reaches U6.10 (SIWU_N)
- net FPGA-F15: now also R199.2
- net FPGA-C22: now reaches U6.11 (WR_N)
- net FPGA-C22: now also R200.2
- net FPGA-F13: now reaches U6.12 (RD_N)
- net FPGA-F13: now also R198.2
- net FPGA-F14: now reaches U6.13 (OE_N)
- net FPGA-F14: now also R197.2
- net FPGA-F16: now reaches U6.15 (RESET_N)
- net FPGA-F16: now also R203.2
- net FPGA-C13: now reaches U6.4 (BE_0)
- net FPGA-C13: now also R193.2
- net FPGA-C14: now reaches U6.5 (BE_1)
- net FPGA-C14: now also R194.2
- net FPGA-C15: now reaches U6.6 (BE_2)
- net FPGA-C15: now also R195.2
- net FPGA-C17: now reaches U6.7 (BE_3)
- net FPGA-C17: now also R196.2
- net FPGA-C19: now reaches U6.8 (TXE_N)
- net FPGA-C19: now also R201.2
- net FPGA-C20: now reaches U6.9 (RXF_N)
- net FPGA-C20: now also R202.2
Other:
- moved on the sheet: R141, R142, R144, R145
