File: 4_Schematics and Boards Layout/4_6_Schematics/MainBoard/RADAR_Main_Board_3.kicad_sch (KiCad schematic)
At the start: 401 parts, among them J20 142-0731-211, J21 CJT-T-P-HH-ST-TH1, J22 142-0731-211, J23 142-0731-211, J24 142-0731-211, J25 142-0731-211, J26 142-0731-211, J27 142-0731-211, J28 142-0731-211, J29 142-0731-211, J30 142-0731-211, J31 142-0731-211, J32 142-0731-211, J33 142-0731-211, J34 142-0731-211, J35 142-0731-211, J36 142-0731-211, J37 142-0731-211, J38 142-0731-211, J39 142-0731-211, J40 142-0731-211, J41 142-0731-211, J42 142-0731-211, J43 142-0731-211, J44 142-0731-211, J45 142-0731-211, J46 142-0731-211, J47 142-0731-211, J48 142-0731-211, J49 142-0731-211, J50 142-0731-211, J51 142-0731-211, J52 142-0731-211, J53 142-0731-211, J54 142-0731-211, J55 142-0731-211, U1 AD9484BCPZ-500, U13 LTC5552IUDBTRMPBF, U14 SZMMSZ5232BT1G, U15 SZMMSZ5232BT1G, U16 EP4RKU+, U17 SZMMSZ5232BT1G, U3 AD9708AR, U37 SZMMSZ5232BT1G, U38 SZMMSZ5232BT1G, U39 SZMMSZ5232BT1G, U4 AD8352ACPZ-R7, U40 SZMMSZ5232BT1G, U41 SZMMSZ5232BT1G, U43 SZMMSZ5232BT1G, U44 SZMMSZ5232BT1G, U45 SZMMSZ5232BT1G, U46 SZMMSZ5232BT1G, U47 SZMMSZ5232BT1G, U48 SZMMSZ5232BT1G, U49 SZMMSZ5232BT1G, U5 LTC5552IUDBTRMPBF, U50 SZMMSZ5232BT1G, U51 SZMMSZ5232BT1G, U52 SZMMSZ5232BT1G, U53 SZMMSZ5232BT1G, U54 SZMMSZ5232BT1G, U55 SZMMSZ5232BT1G, U56 SZMMSZ5232BT1G, U57 SZMMSZ5232BT1G, U58 SZMMSZ5232BT1G, U59 SZMMSZ5232BT1G, U60 SZMMSZ5232BT1G, U61 SZMMSZ5232BT1G, U62 SZMMSZ5232BT1G, U63 SZMMSZ5232BT1G, U64 SZMMSZ5232BT1G, U65 SZMMSZ5232BT1G, U66 SZMMSZ5232BT1G, U67 SZMMSZ5232BT1G, U68 SZMMSZ5232BT1G, U8 AD8352ACPZ-R7

Commit message: KiCad FPGA swap schematic wiring + MCU scan scheduler fix
Manual KiCad work: FPGA swap from XC7A100T to XC7A200T on MainBoard
schematic — rewiring U42 connections, ERC fixes, power rail updates,
PCB footprint swap. Includes backup files and automation scripts.

MCU: scan scheduler contract test + main.cpp updates.
Connections:
- no-connect marks 0 -> 1
Other:
- moved on the sheet: R47, R70, R71, R73, R74, R76, R77

Commit message: FPGA v8c: BRAM playback pipeline with 2048-entry FIFO + USB pipe init fix
- Add unified playback wrapper (radar_system_top_te0713_umft601x_playback.v)
  with BRAM->DSP->USB pipeline, 2048-entry range FIFO, and 3-state
  handshake pop FSM for lossless data delivery to FT601
- Add write_idle output to usb_data_interface.v with fsm_encoding=none
  attributes to prevent Vivado FSM inference bugs
- Add _init_pipes() to radar_protocol.py and ft601_stream_server.py:
  ClearStreamPipe+SetStreamPipe sequence fixes D3XX read timeouts after
  FPGA reprogramming or USB reconnects
- Add Vivado build script, programming script, and 54-test testbench
- KiCad main board schematic wiring progress
- Verified: 2048 range packets delivered end-to-end through full pipeline
  (FPGA->FT601->USB3->stream server->TCP->SSH tunnel->GUI dashboard)
Changed lines of the file:
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@@
 	(symbol
 		(lib_id "RADAR_Main_Board-eagle-import:FRAME_E_L")
-		(at 674.37 787.4 0)
+		(at 576.58 835.66 0)
 		(unit 1)
 		(body_style 1)
@@
 		(dnp no)
 		(property "Reference" "#FRAME3"
-			(at 674.37 787.4 0)
+			(at 576.58 835.66 0)
 			(hide yes)
 			(show_name no)
@@
 		)
 		(property "Value" "FRAME_E_L"
-			(at 674.37 787.4 0)
+			(at 576.58 835.66 0)
 			(hide yes)
 			(show_name no)
@@
 		)
 		(property "Footprint" ""
-			(at 674.37 787.4 0)
+			(at 576.58 835.66 0)
 			(hide yes)
 			(show_name no)
@@
 		)
 		(property "Datasheet" ""
-			(at 674.37 787.4 0)
+			(at 576.58 835.66 0)
 			(hide yes)
 			(show_name no)
@@
 		)
 		(property "Description" "FRAME E Size , 34 x 44 INCH, Landscape"
-			(at 674.37 787.4 0)
+			(at 576.58 835.66 0)
 			(hide yes)
 			(show_name no)
